File: MP1584-5V.kicad_sch (KiCad schematic)
At the start: 15 parts, among them J1 Conn_01x02, J2 Conn_01x02

Commit message: Finalisation PCB
Other:
- title: Janus's 5V DC-DC Buck Converter -> Takes up to 28V and gives 5V as output
Changed lines of the file:
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@@
 	(paper "A4")
 	(title_block
-		(title "Janus's 5V DC-DC Buck Converter")
+		(title "Takes up to 28V and gives 5V as output")
+		(comment 1 "Takes up to 28V and 3A")
+		(comment 2 "This is a 5V DC-DC Buck StepDown converter ")
 	)
 	(junction
